Commit message: Adds dae mesh for finger grippers

File: sisko_mira_description/urdf/r2d2.urdf (robot description, URDF)
Before this commit: robot R2D2, 12 links, 11 joints
Links:
- added link gripper_left_finger; visual mesh filename=package://urdf_tutorial/meshes/l_finger.dae
- added link gripper_left_finger_tip; visual mesh filename=package://urdf_tutorial/meshes/l_finger_tip.dae
- added link gripper_right_finger; visual mesh filename=package://urdf_tutorial/meshes/l_finger.dae
- added link gripper_right_finger_tip; visual mesh filename=package://urdf_tutorial/meshes/l_finger_tip.dae
Joints:
- added joint gripperLeft_finger_tip_to_gripper: type fixed, parent gripper_left_finger, child gripper_left_finger_tip, origin xyz=0.10 0.0 0.0 rpy=0.0 0.0 0.0
- added joint gripperLeft_to_gripper: type fixed, parent gripper_arm, child gripper_left_finger, origin xyz=0.7 0.0 0.15 rpy=0.0 0.0 0.0
- added joint gripperRight_finger_tip_to_gripper: type fixed, parent gripper_right_finger, child gripper_right_finger_tip, origin xyz=0.10 0.0 0.0 rpy=0.0 0.0 0.0
- added joint gripperRight_to_gripper: type fixed, parent gripper_arm, child gripper_right_finger, origin xyz=0.7 -0.0 0.15 rpy=-3.1415 0.0 0.0

Commit message: Fixes wheels and gripper rotation by making joints revolute and adding axis element to joints

File: sisko_mira_description/urdf/r2d2.urdf (robot description, URDF)
Before this commit: robot R2D2, 16 links, 15 joints
Joints:
- joint gripperLeft_to_gripper: axis (none) -> 0.0 0.0 1.0; limit (none) -> lower=0.0 upper=0.548 effort=1000.0 velocity=0.5; type fixed -> revolute
- joint gripperRight_to_gripper: axis (none) -> 0.0 0.0 1.0; limit (none) -> lower=0.0 upper=0.548 effort=1000.0 velocity=0.5; type fixed -> revolute
- joint gripper_arm_joint: limit (none) -> lower=-0.38 upper=0 effort=1000.0 velocity=0.5; type fixed -> prismatic
- joint header_joint: axis (none) -> 0.0 0.0 1.0; type revolute -> continuous
- joint leftbase_front_wheel_joint: axis (none) -> 0.0 1.0 0.0; type revolute -> continuous
- joint leftbase_rear_wheel_joint: axis (none) -> 0.0 1.0 0.0; type revolute -> continuous
- joint rightbase_front_wheel_joint: axis (none) -> 0.0 1.0 0.0; type revolute -> continuous
- joint rightbase_rear_wheel_joint: axis (none) -> 0.0 1.0 0.0; type revolute -> continuous

Commit message: Updated but a work-in-progress. Collision and Inertial tags have not been given to the mesh finger and finger tips link

File: sisko_mira_description/urdf/r2d2.urdf (robot description, URDF)
Before this commit: robot R2D2, 16 links, 15 joints
Links:
- link gripper_arm: mass None -> 10; geometry collision cylinder length=0.5 radius=0.006; visual cylinder length=0.5 radius=0.006
- link headbox: mass None -> 10; geometry collision box size=0.05 0.05 0.05; visual box size=0.05 0.05 0.05
- link header_link: mass None -> 10; geometry collision sphere radius=0.2; visual sphere radius=0.2
- link leftbase_front_wheel: mass None -> 10; geometry collision cylinder length=0.1 radius=0.05; visual cylinder length=0.1 radius=0.05
- link leftbase_rear_wheel: mass None -> 10; geometry collision cylinder length=0.1 radius=0.05; visual cylinder length=0.1 radius=0.05
- link leftleg_base_link: mass None -> 10; geometry collision box size=0.4 0.1 0.1; visual box size=0.4 0.1 0.1
- link leftleg_link: mass None -> 10; geometry collision box size=0.6 0.1 0.2; visual box size=0.6 0.1 0.2
- link rightbase_front_wheel: mass None -> 10; geometry collision cylinder length=0.1 radius=0.05; visual cylinder length=0.1 radius=0.05
- link rightbase_rear_wheel: mass None -> 10; geometry collision cylinder length=0.1 radius=0.05; visual cylinder length=0.1 radius=0.05
- link rightleg_base_link: mass None -> 10; geometry collision box size=0.4 0.1 0.1; visual box size=0.4 0.1 0.1
- link rightleg_link: mass None -> 10; geometry collision box size=0.6 0.1 0.2; visual box size=0.6 0.1 0.2
